Commit message: Enhance simulation setup: update justfile commands, add NEMA 17 motor and parameters xacro files

File: src/armold_description/urdf/armold.urdf.xacro (robot description, xacro)
@@ -9,4 +9,7 @@
 -->
 <robot name="armold" xmlns:xacro="http://www.ros.org/wiki/xacro">
+  <!-- Mass table (edit masses there, not here) and reusable components -->
+  <xacro:include filename="$(find armold_description)/urdf/parameters.xacro"/>
+  <xacro:include filename="$(find armold_description)/urdf/nema17.xacro"/>
   <!-- ================================================================== -->
   <!-- Conversions and shared properties                                   -->
@@ -37,12 +40,6 @@
   <xacro:property name="j1_base_height"     value="${60.750 * mm}"/>
   <xacro:property name="j1_base_top_bore_r" value="${25.000 * mm}"/>
-  <!--
-    Mass is an ESTIMATE, not a measurement: mesh solid volume 61563.1 mm^3
-    (61.563 cm^3) times PLA density, assuming 100% infill. A printed part is not
-    solid, so replace this with a weighed value before doing any dynamics.
-  -->
-  <xacro:property name="pla_density"    value="1240.0"/>            <!-- kg/m^3 -->
-  <xacro:property name="j1_base_volume" value="61.5631e-6"/>        <!-- m^3    -->
-  <xacro:property name="j1_base_mass"   value="${pla_density * j1_base_volume}"/>
+  <!-- Mass lives in the table in parameters.xacro -->
+  <xacro:property name="j1_base_mass" value="${mass_j1_base}"/>
   <!-- ================================================================== -->
   <!-- Materials                                                           -->

Commit message: Add J1 mounting bracket definition and mass parameter to URDF files

File: src/armold_description/urdf/armold.urdf.xacro (robot description, xacro)
@@ -106,7 +106,77 @@
     </inertial>
   </link>
+  <!-- ================================================================== -->
+  <!-- J1 stepper mount - STATIC                                           -->
+  <!-- ================================================================== -->
   <!--
-    NEXT: J1 revolute joint about +Z, mounted on the top face at
-    z = ${j1_base_height} (60.750 mm), carrying "J1 J5 - Mounting Bracket".
+    Source mesh : J1 J5 - Mounting Bracket.stl  (11008 triangles)
+    Measured    : outer edge least-squares fit over 374 rim vertices
+                    centre   (+0.000000, -0.000000) mm  -> 0.00 microns off axis
+                    radius   31.00001 mm  (diameter 62.0000)
+                    rms circularity error 0.0 microns  (exact)
+                  bbox z     0.000 .. 8.050 mm  (a flat disc)
+                  underside  flat annulus r 11.750..30.850 at z = 0, and NOTHING
+                             protrudes below z = 0 - so there is no centring
+                             spigot; the disc simply seats on the base top face.
+                  motor      4 holes at (+/-15.500, +/-15.500) mm = a 31.0 mm
+                             square pattern, dia 3.00 mm, counterbored to
+                             6.50 mm at the top face. That is the NEMA 17
+                             bolt pattern (31.04 mm nominal).
+                  8 x dia 2.10 mm holes on a 56 mm bolt circle (r = 28.000)
+    PLACEMENT: the bracket's underside is flat and its mesh origin is already on
+    the common axis to 0.00 microns, so it needs no offset of its own. The joint
+    simply lifts it to the base's top face at z = 60.750 mm. Mesh used exactly as
+    authored - the geometry is preserved, only the frame moves.
+    THIS PART DOES NOT ROTATE. It is the stepper's mount: it clamps the motor
+    BODY, so it is rigidly part of the static base assembly. The 31.0 mm square
+    hole pattern measured above is what bolts the motor to it. J1's actual
+    rotation is driven by the motor SHAFT, which turns whatever mounts above -
+    so the revolute joint belongs on that next part, not here.
+  -->
+  <xacro:property name="j1_bracket_radius"    value="${31.00001 * mm}"/>
+  <xacro:property name="j1_bracket_thickness" value="${8.050 * mm}"/>
+  <!--
+    Fixed, not revolute: the bracket holds the motor body, so it never moves
+    relative to the base.
+  -->
+  <joint name="base_to_j1_mount" type="fixed">
+    <parent link="base_link"/>
+    <child  link="j1_mounting_bracket"/>
+    <origin xyz="0 0 ${j1_base_height}" rpy="0 0 0"/>
+  </joint>
+  <link name="j1_mounting_bracket">
+    <visual>
+      <!-- mesh authored about this exact frame; used unmodified -->
+      <origin xyz="0 0 0" rpy="0 0 0"/>
+      <geometry>
+        <mesh filename="${mesh_dir}/visual/j1_j5_mounting_bracket.stl"
+              scale="${mesh_scale}"/>
+      </geometry>
+      <material name="armold_black"/>
+    </visual>
+    <!--
+      A cylinder is not an approximation here: the part is a plain disc, so
+      r = 31.000 mm, h = 8.050 mm IS its exact envelope. Only internal pockets
+      and bolt holes are lost, and those cannot participate in a collision.
+    -->
+    <collision>
+      <origin xyz="0 0 ${j1_bracket_thickness / 2}" rpy="0 0 0"/>
+      <geometry>
+        <cylinder radius="${j1_bracket_radius}" length="${j1_bracket_thickness}"/>
+      </geometry>
+    </collision>
+    <inertial>
+      <origin xyz="0 0 ${j1_bracket_thickness / 2}" rpy="0 0 0"/>
+      <mass value="${mass_j1_j5_bracket}"/>
+      <inertia
+        ixx="${mass_j1_j5_bracket * (3 * j1_bracket_radius * j1_bracket_radius + j1_bracket_thickness * j1_bracket_thickness) / 12}"
+        iyy="${mass_j1_j5_bracket * (3 * j1_bracket_radius * j1_bracket_radius + j1_bracket_thickness * j1_bracket_thickness) / 12}"
+        izz="${mass_j1_j5_bracket * j1_bracket_radius * j1_bracket_radius / 2}"
+        ixy="0" ixz="0" iyz="0"/>
+    </inertial>
+  </link>
+  <!--
+    NEXT: the J1 revolute joint itself - about +Z, driven by the motor shaft,
+    carrying whatever mounts on the shaft above this bracket.
   -->
 </robot>

File: src/armold_description/urdf/parameters.xacro (robot description, xacro)
@@ -22,4 +22,9 @@
        recorded for completeness and for shipping-weight sums only. -->
   <xacro:property name="mass_j1_base" value="0.0763"/>
+  <!-- [ESTIMATE] J1/J5 mounting bracket.
+       Mesh solid volume 21 045.9 mm^3 = 21.0459e-6 m^3, x PLA 1240 kg/m^3.
+       Static - it clamps the motor body and is part of the fixed base
+       assembly - so like the base its mass never enters the dynamics. -->
+  <xacro:property name="mass_j1_j5_bracket" value="0.0261"/>
   <!-- ================================================================ -->
   <!-- Motors                                                            -->

Commit message: Add J2 base T-joint definition and mass parameter to URDF files

File: src/armold_description/urdf/armold.urdf.xacro (robot description, xacro)
@@ -176,7 +176,92 @@
     </inertial>
   </link>
-  <!--
-    NEXT: the J1 revolute joint itself - about +Z, driven by the motor shaft,
-    carrying whatever mounts on the shaft above this bracket.
+  <!-- ================================================================== -->
+  <!-- J1 - base rotation about +Z, driven by the stepper shaft             -->
+  <!-- ================================================================== -->
+  <!--
+    Source mesh : J2 - Base T-Joint.stl  (36114 triangles)
+    Measured    : the lower section is a stack of cylinders, every one of them
+                  concentric with the mesh Z axis to 0.0 microns:
+                    z  0.0- 2.0   outer r 31.0000  centre (+0.0000,+0.0000)
+                    z  6.0-12.0   outer r 26.0000  centre (+0.0000,+0.0000)
+                    z 12.0-20.0   outer r 24.4646  centre (-0.0000,-0.0000)
+                  bottom face z=0: annulus r 26.500..30.500, centre (0,0),
+                                   circularity rms 0.0 microns
+                  bbox        x +/-31.000, y -36.000..46.800, z 0..92.000
+                              (asymmetric in Y - that is the T arm)
+    PLACEMENT: the bottom annulus (r 26.500..30.500) seats on the bracket's top
+    face (r 6.750..30.500) - the two rings coincide, so this simply stacks. The
+    mesh's own axis of revolution is already the rotation axis, so once again the
+    mesh is used exactly as authored with no offset or rotation of its own.
+    This is the first link that MOVES: the stepper's shaft turns it about +Z,
+    while the mount below holds the motor body still.
+  -->
+  <xacro:property name="j2_t_joint_seat_r_min" value="${26.500 * mm}"/>
+  <xacro:property name="j2_t_joint_seat_r_max" value="${30.500 * mm}"/>
+  <!--
+    Inertia below is EXACT for the geometry, not a primitive approximation.
+    Computed by decomposing the mesh into tetrahedra and integrating the second
+    moment over the solid (validated against a unit cube to 6 decimal places).
+    Stored per unit mass, so the numbers stay correct when the estimated mass is
+    replaced by a weighed one - only the scale changes, never the shape.
+      centre of mass  (-0.3871, -1.7634, +48.8911) mm
+    The off-diagonal terms are small but real (up to 1.8% of the largest
+    diagonal); they come from the arm being offset in Y, so they are kept.
+  -->
+  <xacro:property name="j2_ixx_per_kg" value="1.332202753e-03"/>
+  <xacro:property name="j2_iyy_per_kg" value="1.142624054e-03"/>
+  <xacro:property name="j2_izz_per_kg" value="9.905486229e-04"/>
+  <xacro:property name="j2_ixy_per_kg" value="1.270531800e-05"/>
+  <xacro:property name="j2_ixz_per_kg" value="4.093846446e-06"/>
+  <xacro:property name="j2_iyz_per_kg" value="2.374568760e-05"/>
+  <!--
+    LIMITS ARE PROVISIONAL: +/-180 deg is a placeholder, not a measured or
+    specified value. Effort and velocity likewise, until the gearing is known.
+  -->
+  <joint name="J1" type="revolute">
+    <parent link="j1_mounting_bracket"/>
+    <child  link="j2_base_t_joint"/>
+    <!-- the bracket's top face, i.e. its own thickness above its frame -->
+    <origin xyz="0 0 ${j1_bracket_thickness}" rpy="0 0 0"/>
+    <axis xyz="0 0 1"/>
+    <limit lower="${-pi}" upper="${pi}" effort="10.0" velocity="3.14"/>
+  </joint>
+  <link name="j2_base_t_joint">
+    <visual>
+      <origin xyz="0 0 0" rpy="0 0 0"/>
+      <geometry>
+        <mesh filename="${mesh_dir}/visual/j2_base_t_joint.stl"
+              scale="${mesh_scale}"/>
+      </geometry>
+      <material name="armold_black"/>
+    </visual>
+    <!--
+      The mesh itself is used for collision. This part is a T, not a solid of
+      revolution, so no primitive is its true envelope and substituting one would
+      throw away exactly the geometry we are trying to preserve. It costs 36114
+      triangles; if collision checking ever gets slow, put a decimated hull in
+      meshes/collision/ and point this at it instead.
+    -->
+    <collision>
+      <origin xyz="0 0 0" rpy="0 0 0"/>
+      <geometry>
+        <mesh filename="${mesh_dir}/visual/j2_base_t_joint.stl"
+              scale="${mesh_scale}"/>
+      </geometry>
+    </collision>
+    <inertial>
+      <origin xyz="${-0.3871 * mm} ${-1.7634 * mm} ${48.8911 * mm}" rpy="0 0 0"/>
+      <mass value="${mass_j2_base_t_joint}"/>
+      <inertia
+        ixx="${mass_j2_base_t_joint * j2_ixx_per_kg}"
+        iyy="${mass_j2_base_t_joint * j2_iyy_per_kg}"
+        izz="${mass_j2_base_t_joint * j2_izz_per_kg}"
+        ixy="${mass_j2_base_t_joint * j2_ixy_per_kg}"
+        ixz="${mass_j2_base_t_joint * j2_ixz_per_kg}"
+        iyz="${mass_j2_base_t_joint * j2_iyz_per_kg}"/>
+    </inertial>
+  </link>
+  <!--
+    NEXT: J2 itself, higher up this T-joint, carrying "J3 J4 - C-Joint".
   -->
 </robot>

File: src/armold_description/urdf/parameters.xacro (robot description, xacro)
@@ -27,4 +27,9 @@
        assembly - so like the base its mass never enters the dynamics. -->
   <xacro:property name="mass_j1_j5_bracket" value="0.0261"/>
+  <!-- [ESTIMATE] J2 base T-joint - the first MOVING link.
+       Mesh solid volume 112 430.4 mm^3 = 112.4304e-6 m^3, x PLA 1240 kg/m^3.
+       This one rotates, so its mass and inertia genuinely matter: it is the
+       entire load the J1 stepper has to accelerate. Weigh it. -->
+  <xacro:property name="mass_j2_base_t_joint" value="0.1394"/>
   <!-- ================================================================ -->
   <!-- Motors                                                            -->

Commit message: Add J1 and J2 motor definitions with mass parameters to URDF files

File: src/armold_description/urdf/armold.urdf.xacro (robot description, xacro)
@@ -176,4 +176,28 @@
     </inertial>
   </link>
+  <!--
+    The J1 stepper, held by the mounting bracket above it. Measured:
+      bolt pattern  4 x dia 3.00 at (+/-15.500, +/-15.500) = 31.0 mm square,
+                    countersunk to dia 6.50 at the bracket's TOP face (z=8.05)
+                    - so the heads sit flush on top and the screws thread DOWN
+                    into the motor underneath.
+      pilot recess  the bracket's bottom face (z=0) has a dia 23.50 central
+                    opening; a NEMA 17's dia 22 boss seats in it.
+      shaft bore    narrows to dia 13.00 higher up - clearance for the shaft,
+                    which passes up through the bracket and drives the T-joint.
+    So the bracket is placed OVER the motor: the motor's mounting face presses
+    against the bracket's underside at z = 0, its body hangs down into the base
+    tube (to z = -37.5 mm, i.e. z = 23.25 in base_link), and the shaft points UP.
+    That is the macro's native frame - mounting face at the origin, +Z along the
+    shaft, body into -Z - so this needs no rotation at all: rpy = 0.
+    This motor is completely enclosed by the base tube. visual is left on because
+    a box costs 12 triangles, and being able to hide base_link and check the
+    motor sits where it should is worth more than that.
+  -->
+  <xacro:nema17 name="j1_motor" parent="j1_mounting_bracket"
+                mass="${mass_nema17_37_5}" body_length="${37.5 * mm}"
+                visual="true" shaft="true">
+    <origin xyz="0 0 0" rpy="0 0 0"/>
+  </xacro:nema17>
   <!-- ================================================================== -->
   <!-- J1 - base rotation about +Z, driven by the stepper shaft             -->
@@ -263,4 +287,32 @@
   </link>
   <!--
+    The J2 stepper, carried by the T-joint. Measured from the mesh:
+      bolt pattern  4 x dia 3.00 mm at (x, z) = (+/-15.500, 45.500)
+                    and (+/-15.500, 76.500) -> a 31.0 x 31.0 mm square in the
+                    XZ plane, so the motor axis runs along Y (not Z).
+                    Pattern centre: x = 0, z = 61.000 mm.
+      plate         flat faces at y = -36.000 (outer) and y = -27.950 (inner),
+                    i.e. 8.05 mm thick.
+      screws        enter at y = -36.000 through a dia 6.50 counterbore, pass
+                    through dia 3.00 clearance, and thread into the motor.
+      pilot         recess at r ~= 11.5-11.75 mm (dia 23) just inside y = -27.950
+                    - that is the seat for the NEMA 17's dia 22 boss.
+      shaft         dia 13.0 clearance hole through the plate at (0, 61).
+    So the motor's mounting face sits against the plate's INNER face at
+    y = -27.950, its body runs in +Y (to y = +32.05 for a 60 mm can, well inside
+    the part's y extent of 46.8), and its shaft points in -Y.
+    The macro's frame is the centre of the mounting face with +Z along the shaft.
+    rpy = (pi/2, 0, 0) rotates that frame's +Z onto -Y, which is where the shaft
+    points; the body then extends along -Z, i.e. +Y. Nothing is scaled or moved
+    by hand - the pose comes straight from the measured face and pattern centre.
+    visual is ON here because the motor sits in the open mouth of the T and is
+    genuinely visible; set it to false if the extra draw ever costs anything.
+  -->
+  <xacro:nema17 name="j2_motor" parent="j2_base_t_joint"
+                mass="${mass_nema17_60}" body_length="${60.0 * mm}"
+                visual="true" shaft="true">
+    <origin xyz="0 ${-27.950 * mm} ${61.000 * mm}" rpy="${pi/2} 0 0"/>
+  </xacro:nema17>
+  <!--
     NEXT: J2 itself, higher up this T-joint, carrying "J3 J4 - C-Joint".
   -->

File: src/armold_description/urdf/parameters.xacro (robot description, xacro)
@@ -40,4 +40,10 @@
        inertia, so WEIGH ONE and replace this before trusting any dynamics. -->
   <xacro:property name="mass_nema17_37_5" value="0.250"/>
+  <!-- [ESTIMATE] NEMA 17, 60 mm body - the J2 motor, carried by the T-joint.
+       A 60 mm can is among the longest NEMA 17s made; catalogue weights run
+       roughly 0.40-0.50 kg, so this is a wide guess. It rides on a moving link
+       AND is the heaviest single item so far - about 3x the T-joint itself - so
+       it dominates the J1 inertia. This is the most valuable part to weigh. -->
+  <xacro:property name="mass_nema17_60" value="0.450"/>
   <!-- ================================================================ -->
   <!-- Material densities (for volume-based estimates)                   -->

Commit message: Add J2 joint definition and mass parameters to URDF files

File: src/armold_description/urdf/armold.urdf.xacro (robot description, xacro)
@@ -314,6 +314,95 @@
     <origin xyz="0 ${-27.950 * mm} ${61.000 * mm}" rpy="${pi/2} 0 0"/>
   </xacro:nema17>
-  <!--
-    NEXT: J2 itself, higher up this T-joint, carrying "J3 J4 - C-Joint".
+  <!-- ================================================================== -->
+  <!-- J2 - shoulder rotation, driven by the 60 mm stepper in the T-joint   -->
+  <!-- ================================================================== -->
+  <!--
+    Source mesh : J3 J4 - C-Joint.stl  (52564 triangles)
+    Measured    : bbox x +/-31.001, y -196.000..31.000, z 0.000..68.500
+                  So in its authored (print) pose it lies on its side: 227 mm
+                  long down -Y, with a collar at the +Y end and a fork at the
+                  far end.
+    HOW WE KNOW WHICH END MATES, and which way up:
+      The +Y end carries a collar whose flat faces are
+        z = 6.800 (r 23.255..30.918)   z = 23.000 (r 23.255..26.000)
+        z = 7.050 (r 23.006..24.500)   z = 22.750 (r 23.006..24.500)
+        z = 10.190 (r 24.026..24.486)  z = 12.283 (r 23.006..23.648)
+      Those are the SAME face heights and the SAME radii, to the micron, as the
+      collar on the bottom of J2 - Base T-Joint. It is one standard rotary
+      interface reused: the C-joint seats on the J2 stepper exactly the way the
+      T-joint seats on the J1 stepper.
+      The far end (y ~ -165) is the fork: a 31.0 mm square NEMA 17 pattern on the
+      z = 0 face and an 8-hole 56 mm bolt circle on the z = 62 face, facing each
+      other across the C - that is where J3 lives.
+    PLACEMENT: by that analogy the collar's z = 0 face seats on the J2 motor
+    plate's OUTER face, measured at y = -36.000 in the T-joint, concentric with
+    the motor at (x = 0, z = 61.000). rpy maps the collar axis (+Z of the mesh)
+    onto -Y, i.e. along the shaft and away from the plate, and puts the arm up
+    +Z. Mesh untouched - the pose is all in the joint.
+  -->
+  <xacro:property name="j2_plate_outer_y" value="${-36.000 * mm}"/>
+  <xacro:property name="j2_axis_z"        value="${61.000 * mm}"/>
+  <!--
+    Exact inertia from tetrahedral integration of the mesh, stored per unit mass
+    (same method as the T-joint, validated against a unit cube).
+      centre of mass  (-0.0233, -94.9246, +22.9492) mm in the MESH frame
+    iyy is ~7x smaller than ixx and izz, which is what a long thin arm should
+    look like: little inertia about its own length, lots about the other two.
+  -->
+  <xacro:property name="j3_ixx_per_kg" value="3.612290951e-03"/>
+  <xacro:property name="j3_iyy_per_kg" value="5.026704008e-04"/>
+  <xacro:property name="j3_izz_per_kg" value="3.752252769e-03"/>
+  <xacro:property name="j3_ixy_per_kg" value="-1.821962233e-06"/>
+  <xacro:property name="j3_ixz_per_kg" value="6.683033126e-07"/>
+  <xacro:property name="j3_iyz_per_kg" value="1.688928696e-04"/>
+  <!--
+    Revolute about the C-joint's own +Z - the blue axis in RViz - which the rpy
+    above deliberately aligns with the stepper shaft. Working it through:
+      Rx(-90) sends (0,0,1) to (0,1,0), then Rz(180) sends that to (0,-1,0),
+    so the child frame's +Z lands on the T-joint's -Y, which is exactly the
+    direction the J2 motor shaft points. In URDF the axis is expressed in the
+    joint (== child) frame, so plain "0 0 1" is the shaft axis.
+    LIMITS ARE PROVISIONAL: +/-180 deg is a placeholder, not a measured or
+    specified value - a real shoulder will hit its own structure long before
+    that. Effort and velocity likewise, until the gearing is known.
+  -->
+  <joint name="J2" type="revolute">
+    <parent link="j2_base_t_joint"/>
+    <child  link="j3_j4_c_joint"/>
+    <origin xyz="0 ${j2_plate_outer_y} ${j2_axis_z}" rpy="${-pi/2} 0 ${pi}"/>
+    <axis xyz="0 0 1"/>
+    <limit lower="${-pi}" upper="${pi}" effort="10.0" velocity="3.14"/>
+  </joint>
+  <link name="j3_j4_c_joint">
+    <visual>
+      <origin xyz="0 0 0" rpy="0 0 0"/>
+      <geometry>
+        <mesh filename="${mesh_dir}/visual/j3_j4_c_joint.stl"
+              scale="${mesh_scale}"/>
+      </geometry>
+      <material name="armold_black"/>
+    </visual>
+    <!-- mesh collision: a C-shaped arm has no meaningful primitive envelope -->
+    <collision>
+      <origin xyz="0 0 0" rpy="0 0 0"/>
+      <geometry>
+        <mesh filename="${mesh_dir}/visual/j3_j4_c_joint.stl"
+              scale="${mesh_scale}"/>
+      </geometry>
+    </collision>
+    <inertial>
+      <origin xyz="${-0.0233 * mm} ${-94.9246 * mm} ${22.9492 * mm}" rpy="0 0 0"/>
+      <mass value="${mass_j3_j4_c_joint}"/>
+      <inertia
+        ixx="${mass_j3_j4_c_joint * j3_ixx_per_kg}"
+        iyy="${mass_j3_j4_c_joint * j3_iyy_per_kg}"
+        izz="${mass_j3_j4_c_joint * j3_izz_per_kg}"
+        ixy="${mass_j3_j4_c_joint * j3_ixy_per_kg}"
+        ixz="${mass_j3_j4_c_joint * j3_ixz_per_kg}"
+        iyz="${mass_j3_j4_c_joint * j3_iyz_per_kg}"/>
+    </inertial>
+  </link>
+  <!--
+    NEXT: make J2 revolute about the shaft axis, then J3 in the C-joint's fork.
   -->
 </robot>

File: src/armold_description/urdf/parameters.xacro (robot description, xacro)
@@ -32,4 +32,9 @@
        entire load the J1 stepper has to accelerate. Weigh it. -->
   <xacro:property name="mass_j2_base_t_joint" value="0.1394"/>
+  <!-- [ESTIMATE] J3/J4 C-joint - the upper arm segment, a MOVING link.
+       Mesh solid volume 275 405.6 mm^3 = 275.4056e-6 m^3, x PLA 1240 kg/m^3.
+       227 mm long, so it swings a long lever arm; both its mass and where that
+       mass sits dominate the J2 torque. Weigh it. -->
+  <xacro:property name="mass_j3_j4_c_joint" value="0.3415"/>
   <!-- ================================================================ -->
   <!-- Motors                                                            -->
