Commit message: Add C-joint definition and mass parameters to URDF files

File: src/armold_description/urdf/armold.urdf.xacro (robot description, xacro)
@@ -12,4 +12,5 @@
   <xacro:include filename="$(find armold_description)/urdf/parameters.xacro"/>
   <xacro:include filename="$(find armold_description)/urdf/nema17.xacro"/>
+  <xacro:include filename="$(find armold_description)/urdf/c_joint.xacro"/>
   <!-- ================================================================== -->
   <!-- Conversions and shared properties                                   -->
@@ -343,17 +344,5 @@
   <xacro:property name="j2_plate_outer_y" value="${-36.000 * mm}"/>
   <xacro:property name="j2_axis_z"        value="${61.000 * mm}"/>
-  <!--
-    Exact inertia from tetrahedral integration of the mesh, stored per unit mass
-    (same method as the T-joint, validated against a unit cube).
-      centre of mass  (-0.0233, -94.9246, +22.9492) mm in the MESH frame
-    iyy is ~7x smaller than ixx and izz, which is what a long thin arm should
-    look like: little inertia about its own length, lots about the other two.
-  -->
-  <xacro:property name="j3_ixx_per_kg" value="3.612290951e-03"/>
-  <xacro:property name="j3_iyy_per_kg" value="5.026704008e-04"/>
-  <xacro:property name="j3_izz_per_kg" value="3.752252769e-03"/>
-  <xacro:property name="j3_ixy_per_kg" value="-1.821962233e-06"/>
-  <xacro:property name="j3_ixz_per_kg" value="6.683033126e-07"/>
-  <xacro:property name="j3_iyz_per_kg" value="1.688928696e-04"/>
+  <!-- geometry, mass distribution and inertia all live in c_joint.xacro -->
   <!--
     Revolute about the C-joint's own +Z - the blue axis in RViz - which the rpy
@@ -374,35 +363,54 @@
     <limit lower="${-pi}" upper="${pi}" effort="10.0" velocity="3.14"/>
   </joint>
-  <link name="j3_j4_c_joint">
-    <visual>
-      <origin xyz="0 0 0" rpy="0 0 0"/>
-      <geometry>
-        <mesh filename="${mesh_dir}/visual/j3_j4_c_joint.stl"
-              scale="${mesh_scale}"/>
-      </geometry>
-      <material name="armold_black"/>
-    </visual>
-    <!-- mesh collision: a C-shaped arm has no meaningful primitive envelope -->
-    <collision>
-      <origin xyz="0 0 0" rpy="0 0 0"/>
-      <geometry>
-        <mesh filename="${mesh_dir}/visual/j3_j4_c_joint.stl"
-              scale="${mesh_scale}"/>
-      </geometry>
-    </collision>
-    <inertial>
-      <origin xyz="${-0.0233 * mm} ${-94.9246 * mm} ${22.9492 * mm}" rpy="0 0 0"/>
-      <mass value="${mass_j3_j4_c_joint}"/>
-      <inertia
-        ixx="${mass_j3_j4_c_joint * j3_ixx_per_kg}"
-        iyy="${mass_j3_j4_c_joint * j3_iyy_per_kg}"
-        izz="${mass_j3_j4_c_joint * j3_izz_per_kg}"
-        ixy="${mass_j3_j4_c_joint * j3_ixy_per_kg}"
-        ixz="${mass_j3_j4_c_joint * j3_ixz_per_kg}"
-        iyz="${mass_j3_j4_c_joint * j3_iyz_per_kg}"/>
-    </inertial>
-  </link>
-  <!--
-    NEXT: make J2 revolute about the shaft axis, then J3 in the C-joint's fork.
+  <xacro:c_joint_link name="j3_j4_c_joint" mass="${mass_j3_j4_c_joint}"/>
+  <!-- ================================================================== -->
+  <!-- J3 - elbow, in the first C-joint's fork                              -->
+  <!-- ================================================================== -->
+  <!--
+    The fork's bottom arm is the J1 mounting bracket's interface MIRRORED. Laid
+    side by side, in each part's own frame:
+        bracket                        C-joint fork
+        z = 0     motor face,          z = 8.050  motor face,
+                  dia 23 pilot recess             dia 23 pilot recess (z 6..8.05)
+        z = 3.0   dia 13 shaft bore    z = 0..6   dia 13 shaft bore
+        z = 8.050 collar seat face,    z = 0      collar seat face,
+                  r 6.750..30.500                 r 6.750..30.500
+    Same numbers, opposite order. So the J3 stepper mounts against z = 8.050 with
+    its body reaching UP into the fork's gap, its shaft pointing DOWN, and the
+    next segment's collar seats on the z = 0 face - exactly how the T-joint seats
+    on the bracket at J1.
+  -->
+  <!--
+    Motor: rpy = (pi, 0, 0) turns the macro's +Z (the shaft) onto the parent's
+    -Z, which is where the shaft points; the body then extends along the parent's
+    +Z, up into the gap between the fork's two arms.
+  -->
+  <xacro:nema17 name="j3_motor" parent="j3_j4_c_joint"
+                mass="${mass_nema17_37_5}" body_length="${37.5 * mm}"
+                visual="true" shaft="true">
+    <origin xyz="0 ${c_fork_axis_y} ${c_fork_motor_z}" rpy="${pi} 0 0"/>
+  </xacro:nema17>
+  <!--
+    J3 itself. rpy = (pi, 0, pi) composes to diag(-1, 1, -1), which sends the
+    child's +Z onto the parent's -Z - so the second segment's collar seats on the
+    z = 0 face and extends downward away from it, and its arm carries on in the
+    parent's -Y rather than folding back. As with J1 and J2 the axis is the
+    child's own +Z, the blue axis in RViz.
+    Because J3's axis is the parent's Z and J2's axis was also a Z of this same
+    link, J2 and J3 come out parallel - which is what a shoulder and elbow in a
+    planar arm should be, and a useful check that the chain is right.
+    LIMITS ARE PROVISIONAL: +/-180 deg placeholder, as for J1 and J2.
+  -->
+  <joint name="J3" type="revolute">
+    <parent link="j3_j4_c_joint"/>
+    <child  link="j3_j4_c_joint_2"/>
+    <origin xyz="0 ${c_fork_axis_y} ${c_fork_seat_z}" rpy="${pi} 0 ${pi}"/>
+    <axis xyz="0 0 1"/>
+    <limit lower="${-pi}" upper="${pi}" effort="10.0" velocity="3.14"/>
+  </joint>
+  <!-- the same part again - identical geometry, mass and inertia by construction -->
+  <xacro:c_joint_link name="j3_j4_c_joint_2" mass="${mass_j3_j4_c_joint}"/>
+  <!--
+    NEXT: J4 in the second C-joint's fork, then J5.
   -->
 </robot>

Commit message: Update material definitions in URDF files for improved color accuracy

File: src/armold_description/urdf/armold.urdf.xacro (robot description, xacro)
@@ -46,6 +46,14 @@
   <!-- Materials                                                           -->
   <!-- ================================================================== -->
-  <material name="armold_black">
-    <color rgba="0.15 0.15 0.17 1.0"/>
+  <!--
+    Palette matches the physical print: grey filament throughout, with the
+    mounting bracket in blue. Motors keep their own darker steel grey, defined
+    in nema17.xacro - they are bought parts, not printed.
+  -->
+  <material name="armold_grey">
+    <color rgba="0.62 0.62 0.64 1.0"/>
+  </material>
+  <material name="armold_blue">
+    <color rgba="0.11 0.35 0.72 1.0"/>
   </material>
   <!-- ================================================================== -->
@@ -82,5 +90,5 @@
               scale="${mesh_scale}"/>
       </geometry>
-      <material name="armold_black"/>
+      <material name="armold_grey"/>
     </visual>
     <!--
@@ -154,5 +162,5 @@
               scale="${mesh_scale}"/>
       </geometry>
-      <material name="armold_black"/>
+      <material name="armold_blue"/>
     </visual>
     <!--
@@ -259,5 +267,5 @@
               scale="${mesh_scale}"/>
       </geometry>
-      <material name="armold_black"/>
+      <material name="armold_grey"/>
     </visual>
     <!--

File: src/armold_description/urdf/c_joint.xacro (robot description, xacro)
@@ -42,5 +42,5 @@
           <mesh filename="${mesh_dir}/visual/j3_j4_c_joint.stl" scale="${mesh_scale}"/>
         </geometry>
-        <material name="armold_black"/>
+        <material name="armold_grey"/>
       </visual>
       <!-- mesh collision: a C-shaped arm has no meaningful primitive envelope -->

Commit message: Refactor C-joint definitions for clarity and consistency in URDF files

File: src/armold_description/urdf/armold.urdf.xacro (robot description, xacro)
@@ -366,10 +366,11 @@
   <joint name="J2" type="revolute">
     <parent link="j2_base_t_joint"/>
-    <child  link="j3_j4_c_joint"/>
+    <child  link="j3_c_joint"/>
     <origin xyz="0 ${j2_plate_outer_y} ${j2_axis_z}" rpy="${-pi/2} 0 ${pi}"/>
     <axis xyz="0 0 1"/>
     <limit lower="${-pi}" upper="${pi}" effort="10.0" velocity="3.14"/>
   </joint>
-  <xacro:c_joint_link name="j3_j4_c_joint" mass="${mass_j3_j4_c_joint}"/>
+  <xacro:c_joint_link name="j3_c_joint" mesh="j3_c_joint.stl"
+                      mass="${mass_c_joint}"/>
   <!-- ================================================================== -->
   <!-- J3 - elbow, in the first C-joint's fork                              -->
@@ -394,5 +395,5 @@
     +Z, up into the gap between the fork's two arms.
   -->
-  <xacro:nema17 name="j3_motor" parent="j3_j4_c_joint"
+  <xacro:nema17 name="j3_motor" parent="j3_c_joint"
                 mass="${mass_nema17_37_5}" body_length="${37.5 * mm}"
                 visual="true" shaft="true">
@@ -411,6 +412,6 @@
   -->
   <joint name="J3" type="revolute">
-    <parent link="j3_j4_c_joint"/>
-    <child  link="j3_j4_c_joint_2"/>
+    <parent link="j3_c_joint"/>
+    <child  link="j4_c_joint"/>
     <origin xyz="0 ${c_fork_axis_y} ${c_fork_seat_z}" rpy="${pi} 0 ${pi}"/>
     <axis xyz="0 0 1"/>
@@ -418,7 +419,23 @@
   </joint>
   <!-- the same part again - identical geometry, mass and inertia by construction -->
-  <xacro:c_joint_link name="j3_j4_c_joint_2" mass="${mass_j3_j4_c_joint}"/>
-  <!--
-    NEXT: J4 in the second C-joint's fork, then J5.
+  <xacro:c_joint_link name="j4_c_joint" mesh="j4_c_joint.stl"
+                      mass="${mass_c_joint}"/>
+  <!-- ================================================================== -->
+  <!-- J4 motor - in the second C-joint's fork                              -->
+  <!-- ================================================================== -->
+  <!--
+    Identical part, so identical mounting geometry: face at z = 8.050 with the
+    dia 23 pilot recess above it, body reaching up into the fork gap, shaft
+    pointing down through the dia 13 bore to the collar seat at z = 0. The
+    constants come from c_joint.xacro, so this needs no new measurements - if
+    that interface is ever re-measured, J3 and J4 both follow automatically.
+  -->
+  <xacro:nema17 name="j4_motor" parent="j4_c_joint"
+                mass="${mass_nema17_37_5}" body_length="${37.5 * mm}"
+                visual="true" shaft="true">
+    <origin xyz="0 ${c_fork_axis_y} ${c_fork_motor_z}" rpy="${pi} 0 0"/>
+  </xacro:nema17>
+  <!--
+    NEXT: J4 itself, then J5.
   -->
 </robot>

File: src/armold_description/urdf/c_joint.xacro (robot description, xacro)
@@ -2,7 +2,11 @@
 <!--
   J3/J4 C-Joint - the reusable arm segment.
-  Armold uses this identical part twice: once driven by J2 (hosting J3 in its
-  fork) and once driven by J3 (hosting J4). Emitting both from one macro means
-  the geometry, mass and inertia can never drift apart between instances.
+  Armold uses this identical part twice: once hosting J3's motor in its fork and
+  once hosting J4's. Emitting both from one macro means the geometry, mass and
+  inertia can never drift apart between instances.
+  The two instances point at separate mesh files - j3_c_joint.stl and
+  j4_c_joint.stl - which are byte-identical copies of the one supplied part. The
+  duplication is deliberate: naming each file for the joint it serves keeps the
+  model readable, and the meshes are git-ignored so it costs nothing in the repo.
   The mesh is used exactly as authored - no scale beyond mm->m, no offset, no
   baked-in rotation. Every instance differs only by the joint that positions it.
@@ -32,13 +36,14 @@
   <!--
     name    link name to create
+    mesh    file name inside meshes/visual (j3_c_joint.stl or j4_c_joint.stl)
     mass    kg, from the mass table
     Creates only the link; the caller supplies the joint that places it.
   -->
-  <xacro:macro name="c_joint_link" params="name mass">
+  <xacro:macro name="c_joint_link" params="name mesh mass">
     <link name="${name}">
       <visual>
         <origin xyz="0 0 0" rpy="0 0 0"/>
         <geometry>
-          <mesh filename="${mesh_dir}/visual/j3_j4_c_joint.stl" scale="${mesh_scale}"/>
+          <mesh filename="${mesh_dir}/visual/${mesh}" scale="${mesh_scale}"/>
         </geometry>
         <material name="armold_grey"/>
@@ -48,5 +53,5 @@
         <origin xyz="0 0 0" rpy="0 0 0"/>
         <geometry>
-          <mesh filename="${mesh_dir}/visual/j3_j4_c_joint.stl" scale="${mesh_scale}"/>
+          <mesh filename="${mesh_dir}/visual/${mesh}" scale="${mesh_scale}"/>
         </geometry>
       </collision>

File: src/armold_description/urdf/parameters.xacro (robot description, xacro)
@@ -32,9 +32,9 @@
        entire load the J1 stepper has to accelerate. Weigh it. -->
   <xacro:property name="mass_j2_base_t_joint" value="0.1394"/>
-  <!-- [ESTIMATE] J3/J4 C-joint - the upper arm segment, a MOVING link.
+  <!-- [ESTIMATE] C-joint - the arm segment used twice, at J3 and at J4.
        Mesh solid volume 275 405.6 mm^3 = 275.4056e-6 m^3, x PLA 1240 kg/m^3.
        227 mm long, so it swings a long lever arm; both its mass and where that
        mass sits dominate the J2 torque. Weigh it. -->
-  <xacro:property name="mass_j3_j4_c_joint" value="0.3415"/>
+  <xacro:property name="mass_c_joint" value="0.3415"/>
   <!-- ================================================================ -->
   <!-- Motors                                                            -->

Commit message: Add J4 joint definition and J5 J-joint mass parameter to URDF files

File: src/armold_description/urdf/armold.urdf.xacro (robot description, xacro)
@@ -436,6 +436,79 @@
     <origin xyz="0 ${c_fork_axis_y} ${c_fork_motor_z}" rpy="${pi} 0 0"/>
   </xacro:nema17>
-  <!--
-    NEXT: J4 itself, then J5.
+  <!-- ================================================================== -->
+  <!-- J4 - wrist pitch, driven by the stepper in the second C-joint's fork  -->
+  <!-- ================================================================== -->
+  <!--
+    Source mesh : J5 - J-Joint.stl  (38606 triangles)
+    Measured    : bbox x +/-31.005, y -75.750..31.000, z 0.000..66.000
+    WHY IT MOUNTS THE SAME WAY AS THE C-JOINT:
+      Its +Y end carries the identical rotary collar. Face heights and inner
+      radii, measured on both parts:
+        J-joint   z 6.800 / 7.050 / 10.190 / 12.284 / 13.330 / 16.470 / 22.750 / 23.000
+        C-joint   z 6.800 / 7.050 / 10.190 / 12.283 / 13.330 / 16.470 / 22.750 / 23.000
+        inner r   23.255 / 23.006 / 24.026 / 23.006 / 24.026 / 24.026 / 23.006 / 23.255
+      Same interface to the micron, so it seats on the fork's z = 0 collar face
+      exactly as the C-joint does one joint below. That makes the placement a
+      copy of J3's, not a new derivation.
+    ALSO MEASURED, for the step after this one: 8 x dia 3.30 holes on a 56 mm
+    bolt circle (r = 28.000) with their axis along Y, centred at (x 0, z 35.000).
+    That is where the second "J1 J5 - Mounting Bracket" bolts on to carry J5's
+    motor - the same 56 mm interface the bracket uses at J1.
+  -->
+  <xacro:property name="j5_bracket_circle_z" value="${35.000 * mm}"/>
+  <!--
+    Exact inertia, tetrahedral integration over the mesh, stored per unit mass.
+      centre of mass  (-0.0711, -27.7630, +27.4964) mm in the mesh frame
+  -->
+  <xacro:property name="j5_ixx_per_kg" value="1.097011592e-03"/>
+  <xacro:property name="j5_iyy_per_kg" value="6.819946309e-04"/>
+  <xacro:property name="j5_izz_per_kg" value="1.220726909e-03"/>
+  <xacro:property name="j5_ixy_per_kg" value="-1.287485109e-06"/>
+  <xacro:property name="j5_ixz_per_kg" value="1.128303868e-06"/>
+  <xacro:property name="j5_iyz_per_kg" value="2.200239253e-04"/>
+  <!--
+    Revolute about the child's own +Z - the blue axis in RViz - exactly as at J3,
+    because the fork interface is the same one. rpy = (pi, 0, pi) composes to
+    diag(-1, 1, -1), sending the child's +Z onto the parent's -Z, which is the
+    direction the J4 stepper's shaft points.
+    J2, J3 and J4 therefore all end up parallel. That is correct for this arm:
+    they are the shoulder, elbow and wrist pitch of a planar chain, and only J1
+    (base yaw) and later J5/J6 break that plane.
+    LIMITS ARE PROVISIONAL: +/-180 deg placeholder, as for J1-J3. The J-joint
+    will foul the fork's own arms well before that.
+  -->
+  <joint name="J4" type="revolute">
+    <parent link="j4_c_joint"/>
+    <child  link="j5_j_joint"/>
+    <origin xyz="0 ${c_fork_axis_y} ${c_fork_seat_z}" rpy="${pi} 0 ${pi}"/>
+    <axis xyz="0 0 1"/>
+    <limit lower="${-pi}" upper="${pi}" effort="10.0" velocity="3.14"/>
+  </joint>
+  <link name="j5_j_joint">
+    <visual>
+      <origin xyz="0 0 0" rpy="0 0 0"/>
+      <geometry>
+        <mesh filename="${mesh_dir}/visual/j5_j_joint.stl" scale="${mesh_scale}"/>
+      </geometry>
+      <material name="armold_grey"/>
+    </visual>
+    <collision>
+      <origin xyz="0 0 0" rpy="0 0 0"/>
+      <geometry>
+        <mesh filename="${mesh_dir}/visual/j5_j_joint.stl" scale="${mesh_scale}"/>
+      </geometry>
+    </collision>
+    <inertial>
+      <origin xyz="${-0.0711 * mm} ${-27.7630 * mm} ${27.4964 * mm}" rpy="0 0 0"/>
+      <mass value="${mass_j5_j_joint}"/>
+      <inertia
+        ixx="${mass_j5_j_joint * j5_ixx_per_kg}" iyy="${mass_j5_j_joint * j5_iyy_per_kg}"
+        izz="${mass_j5_j_joint * j5_izz_per_kg}" ixy="${mass_j5_j_joint * j5_ixy_per_kg}"
+        ixz="${mass_j5_j_joint * j5_ixz_per_kg}" iyz="${mass_j5_j_joint * j5_iyz_per_kg}"/>
+    </inertial>
+  </link>
+  <!--
+    NEXT: make J4 revolute, then the J5 mounting bracket + motor on the 56 mm
+    circle, then J6 - Top T-Joint.
   -->
 </robot>

File: src/armold_description/urdf/parameters.xacro (robot description, xacro)
@@ -37,4 +37,9 @@
        mass sits dominate the J2 torque. Weigh it. -->
   <xacro:property name="mass_c_joint" value="0.3415"/>
+  <!-- [ESTIMATE] J5 J-joint - carries the wrist. A MOVING link.
+       Mesh solid volume 91 126.9 mm^3 = 91.1269e-6 m^3, x PLA 1240 kg/m^3.
+       Sits at the far end of the arm, so its mass acts on the longest lever of
+       anything so far - it matters to J2 and J3 more than to J4. Weigh it. -->
+  <xacro:property name="mass_j5_j_joint" value="0.1130"/>
   <!-- ================================================================ -->
   <!-- Motors                                                            -->
