Commit message: Add J1 and J5 mounting brackets with mass parameters to URDF files

File: src/armold_description/urdf/armold.urdf.xacro (robot description, xacro)
@@ -13,4 +13,5 @@
   <xacro:include filename="$(find armold_description)/urdf/nema17.xacro"/>
   <xacro:include filename="$(find armold_description)/urdf/c_joint.xacro"/>
+  <xacro:include filename="$(find armold_description)/urdf/bracket.xacro"/>
   <!-- ================================================================== -->
   <!-- Conversions and shared properties                                   -->
@@ -154,35 +155,6 @@
     <origin xyz="0 0 ${j1_base_height}" rpy="0 0 0"/>
   </joint>
-  <link name="j1_mounting_bracket">
-    <visual>
-      <!-- mesh authored about this exact frame; used unmodified -->
-      <origin xyz="0 0 0" rpy="0 0 0"/>
-      <geometry>
-        <mesh filename="${mesh_dir}/visual/j1_j5_mounting_bracket.stl"
-              scale="${mesh_scale}"/>
-      </geometry>
-      <material name="armold_blue"/>
-    </visual>
-    <!--
-      A cylinder is not an approximation here: the part is a plain disc, so
-      r = 31.000 mm, h = 8.050 mm IS its exact envelope. Only internal pockets
-      and bolt holes are lost, and those cannot participate in a collision.
-    -->
-    <collision>
-      <origin xyz="0 0 ${j1_bracket_thickness / 2}" rpy="0 0 0"/>
-      <geometry>
-        <cylinder radius="${j1_bracket_radius}" length="${j1_bracket_thickness}"/>
-      </geometry>
-    </collision>
-    <inertial>
-      <origin xyz="0 0 ${j1_bracket_thickness / 2}" rpy="0 0 0"/>
-      <mass value="${mass_j1_j5_bracket}"/>
-      <inertia
-        ixx="${mass_j1_j5_bracket * (3 * j1_bracket_radius * j1_bracket_radius + j1_bracket_thickness * j1_bracket_thickness) / 12}"
-        iyy="${mass_j1_j5_bracket * (3 * j1_bracket_radius * j1_bracket_radius + j1_bracket_thickness * j1_bracket_thickness) / 12}"
-        izz="${mass_j1_j5_bracket * j1_bracket_radius * j1_bracket_radius / 2}"
-        ixy="0" ixz="0" iyz="0"/>
-    </inertial>
-  </link>
+  <xacro:bracket_link name="j1_mounting_bracket" mesh="j1_mounting_bracket.stl"
+                      mass="${mass_bracket}"/>
   <!--
     The J1 stepper, held by the mounting bracket above it. Measured:
@@ -508,7 +480,39 @@
     </inertial>
   </link>
-  <!--
-    NEXT: make J4 revolute, then the J5 mounting bracket + motor on the 56 mm
-    circle, then J6 - Top T-Joint.
+  <!-- ================================================================== -->
+  <!-- J5 stepper mount - STATIC, bolted to the J-joint                     -->
+  <!-- ================================================================== -->
+  <!--
+    Measured on the J-joint:
+      face        y = -75.750, r 25.000..31.000 about (x 0, z 35.000)
+      bolt circle 8 x dia 3.30 at r = 28.000, same centre, axis along Y
+    That face is the same interface the base's top uses at J1 - identical radii,
+    identical 56 mm circle - so the same bracket bolts on the same way. Its
+    z = 0 motor face presses against y = -75.750, its body-side cavity faces back
+    into the J-joint, and rpy = (pi/2, 0, 0) turns the bracket's +Z onto the
+    J-joint's -Y so the shaft points outward, away from the arm.
+  -->
+  <xacro:property name="j5_bracket_face_y" value="${-75.750 * mm}"/>
+  <joint name="j5_mount_fixed" type="fixed">
+    <parent link="j5_j_joint"/>
+    <child  link="j5_mounting_bracket"/>
+    <origin xyz="0 ${j5_bracket_face_y} ${j5_bracket_circle_z}" rpy="${pi/2} 0 0"/>
+  </joint>
+  <xacro:bracket_link name="j5_mounting_bracket" mesh="j5_mounting_bracket.stl"
+                      mass="${mass_bracket}"/>
+  <!--
+    The J5 stepper - a 23 mm "pancake" NEMA 17. Same relationship as at J1: the
+    bracket is placed over the motor, so the motor's face presses on the
+    bracket's z = 0 and its body hangs into the cavity behind, shaft pointing up
+    through the bracket to drive whatever seats on z = 8.050. That is the macro's
+    native frame, so rpy = 0.
+  -->
+  <xacro:nema17 name="j5_motor" parent="j5_mounting_bracket"
+                mass="${mass_nema17_23}" body_length="${23.0 * mm}"
+                visual="true" shaft="true">
+    <origin xyz="0 0 0" rpy="0 0 0"/>
+  </xacro:nema17>
+  <!--
+    NEXT: J5 itself, then J6 - Top T-Joint, then the gripper.
   -->
 </robot>

File: src/armold_description/urdf/parameters.xacro (robot description, xacro)
@@ -22,9 +22,9 @@
        recorded for completeness and for shipping-weight sums only. -->
   <xacro:property name="mass_j1_base" value="0.0763"/>
-  <!-- [ESTIMATE] J1/J5 mounting bracket.
+  <!-- [ESTIMATE] Mounting bracket - the stepper mount used at J1 and again at J5.
        Mesh solid volume 21 045.9 mm^3 = 21.0459e-6 m^3, x PLA 1240 kg/m^3.
        Static - it clamps the motor body and is part of the fixed base
        assembly - so like the base its mass never enters the dynamics. -->
-  <xacro:property name="mass_j1_j5_bracket" value="0.0261"/>
+  <xacro:property name="mass_bracket" value="0.0261"/>
   <!-- [ESTIMATE] J2 base T-joint - the first MOVING link.
        Mesh solid volume 112 430.4 mm^3 = 112.4304e-6 m^3, x PLA 1240 kg/m^3.
@@ -56,4 +56,8 @@
        it dominates the J1 inertia. This is the most valuable part to weigh. -->
   <xacro:property name="mass_nema17_60" value="0.450"/>
+  <!-- [ESTIMATE] NEMA 17, 23 mm body - the J5 wrist motor. A short "pancake"
+       NEMA 17; catalogue weights are around 0.13-0.17 kg. It rides at the far
+       end of the arm, so its mass acts on the longest lever in the machine. -->
+  <xacro:property name="mass_nema17_23" value="0.150"/>
   <!-- ================================================================ -->
   <!-- Material densities (for volume-based estimates)                   -->

Commit message: Add J5 joint definition and J6 top T-joint mass parameter to URDF files

File: src/armold_description/urdf/armold.urdf.xacro (robot description, xacro)
@@ -513,6 +513,65 @@
     <origin xyz="0 0 0" rpy="0 0 0"/>
   </xacro:nema17>
-  <!--
-    NEXT: J5 itself, then J6 - Top T-Joint, then the gripper.
+  <!-- ================================================================== -->
+  <!-- J5 - wrist roll, driven by the 23 mm stepper in the J5 bracket       -->
+  <!-- ================================================================== -->
+  <!--
+    Source mesh : J6 - Top T-Joint.stl  (39832 triangles)
+    Measured    : bbox x +/-31.000, y -36.000..33.500, z 0.000..92.000
+                  bottom face z = 0: annulus r 26.500..30.500, outer edge fits a
+                  circle centred (-0.00000, +0.00000) with rms 0.0 microns
+                  collar faces z = 6.800 / 7.050 / 10.190 / 12.283 / 13.330 /
+                                 16.470 / 22.750 / 23.000
+    Those collar faces and radii are IDENTICAL to J2 - Base T-Joint's, so this
+    part seats on the J5 bracket exactly as the base T-joint seats on the J1
+    bracket: its z = 0 annulus on the bracket's z = 8.050 collar seat, turned by
+    the shaft coming up through the bracket. Same interface, same placement,
+    same axis - no new derivation, and the mesh is used exactly as authored.
+    LIMITS ARE PROVISIONAL: +/-180 deg placeholder, as for J1-J4.
+  -->
+  <joint name="J5" type="revolute">
+    <parent link="j5_mounting_bracket"/>
+    <child  link="j6_top_t_joint"/>
+    <origin xyz="0 0 ${brk_seat_z}" rpy="0 0 0"/>
+    <axis xyz="0 0 1"/>
+    <limit lower="${-pi}" upper="${pi}" effort="10.0" velocity="3.14"/>
+  </joint>
+  <!--
+    Exact inertia, tetrahedral integration over the mesh, per unit mass.
+      centre of mass (+0.7584, -5.6073, +47.3052) mm in the mesh frame
+    The off-diagonals are larger here than on the other parts because the T arm
+    is offset in both X and Y; they are kept rather than zeroed.
+  -->
+  <xacro:property name="j6_ixx_per_kg" value="1.262019184e-03"/>
+  <xacro:property name="j6_iyy_per_kg" value="1.167925485e-03"/>
+  <xacro:property name="j6_izz_per_kg" value="8.901849246e-04"/>
+  <xacro:property name="j6_ixy_per_kg" value="-9.711467507e-06"/>
+  <xacro:property name="j6_ixz_per_kg" value="-1.102464757e-05"/>
+  <xacro:property name="j6_iyz_per_kg" value="7.675716812e-05"/>
+  <link name="j6_top_t_joint">
+    <visual>
+      <origin xyz="0 0 0" rpy="0 0 0"/>
+      <geometry>
+        <mesh filename="${mesh_dir}/visual/j6_top_t_joint.stl" scale="${mesh_scale}"/>
+      </geometry>
+      <material name="armold_grey"/>
+    </visual>
+    <collision>
+      <origin xyz="0 0 0" rpy="0 0 0"/>
+      <geometry>
+        <mesh filename="${mesh_dir}/visual/j6_top_t_joint.stl" scale="${mesh_scale}"/>
+      </geometry>
+    </collision>
+    <inertial>
+      <origin xyz="${0.7584 * mm} ${-5.6073 * mm} ${47.3052 * mm}" rpy="0 0 0"/>
+      <mass value="${mass_j6_top_t_joint}"/>
+      <inertia
+        ixx="${mass_j6_top_t_joint * j6_ixx_per_kg}" iyy="${mass_j6_top_t_joint * j6_iyy_per_kg}"
+        izz="${mass_j6_top_t_joint * j6_izz_per_kg}" ixy="${mass_j6_top_t_joint * j6_ixy_per_kg}"
+        ixz="${mass_j6_top_t_joint * j6_ixz_per_kg}" iyz="${mass_j6_top_t_joint * j6_iyz_per_kg}"/>
+    </inertial>
+  </link>
+  <!--
+    NEXT: J6 itself - its motor lives in this top T-joint - then the gripper.
   -->
 </robot>

File: src/armold_description/urdf/parameters.xacro (robot description, xacro)
@@ -42,4 +42,8 @@
        anything so far - it matters to J2 and J3 more than to J4. Weigh it. -->
   <xacro:property name="mass_j5_j_joint" value="0.1130"/>
+  <!-- [ESTIMATE] J6 top T-joint - the wrist body, a MOVING link and the last
+       structural part before the gripper.
+       Mesh solid volume 98 894.2 mm^3 = 98.8942e-6 m^3, x PLA 1240 kg/m^3. -->
+  <xacro:property name="mass_j6_top_t_joint" value="0.1226"/>
   <!-- ================================================================ -->
   <!-- Motors                                                            -->

Commit message: Add J6 motor definition in the top T-joint with detailed measurements

File: src/armold_description/urdf/armold.urdf.xacro (robot description, xacro)
@@ -573,5 +573,29 @@
   </link>
   <!--
-    NEXT: J6 itself - its motor lives in this top T-joint - then the gripper.
+    The J6 stepper - a 23 mm NEMA 17 - in the top T-joint.
+    Measured on J6 - Top T-Joint.stl, and it comes out IDENTICAL to the base
+    T-joint's motor pocket, number for number:
+      bolt pattern  4 x dia 3.00 at (x, z) = (+/-15.500, 45.500) and
+                    (+/-15.500, 76.500) -> 31.0 mm square, centre (0, 61.000)
+      plate         flat faces at y = -36.000 (outer) and y = -27.950 (inner)
+      screws        dia 6.50 counterbore at y = -36.000, dia 3.00 clearance
+      pilot         dia 23.00 / 23.50 recess at y -29.0..-27.0 - the NEMA 17
+                    dia 22 boss seat
+      shaft         dia 13.00 clearance bore through the plate
+    Same part family, same pocket: so the pose is the same as j2_motor's, with
+    only the body length differing (23 mm here against 60 mm at J2). Mounting
+    face y = -27.950, body running +Y, shaft pointing -Y; rpy = (pi/2, 0, 0)
+    turns the macro's +Z onto -Y.
+    Body then spans y -27.950..-4.950, comfortably inside the part's -36.000
+    to +33.500 extent.
+  -->
+  <xacro:nema17 name="j6_motor" parent="j6_top_t_joint"
+                mass="${mass_nema17_23}" body_length="${23.0 * mm}"
+                visual="true" shaft="true">
+    <origin xyz="0 ${-27.950 * mm} ${61.000 * mm}" rpy="${pi/2} 0 0"/>
+  </xacro:nema17>
+  <!--
+    NEXT: J6 itself - the rotation this motor drives - and the Micro Gripper
+    MK II that mounts on it.
   -->
 </robot>

Commit message: Add J6 joint and gripper connection definitions with mass parameters to URDF files

File: src/armold_description/urdf/armold.urdf.xacro (robot description, xacro)
@@ -595,7 +595,69 @@
     <origin xyz="0 ${-27.950 * mm} ${61.000 * mm}" rpy="${pi/2} 0 0"/>
   </xacro:nema17>
-  <!--
-    NEXT: J6 itself - the rotation this motor drives - and the Micro Gripper
-    MK II that mounts on it.
+  <!-- ================================================================== -->
+  <!-- J6 - carries the gripper connection. STATIC FOR NOW.                 -->
+  <!-- ================================================================== -->
+  <!--
+    Source mesh : Gripper - Connection.stl  (27357 triangles)
+    Measured    : bbox x +/-31.000, y +/-31.000, z 0.005..31.905
+                  bottom face z = 0.005: outer edge fits a circle centred
+                  (-0.00000, +0.00000), r = 30.5000, rms 0.0 microns
+                  central bore dia 4.15..4.74 running z 0..18 - not round: the
+                  radius drops to 2.075 on one side and sits at ~2.37 elsewhere,
+                  which is a D-bore for the NEMA 17's dia 5 flatted shaft.
+    HOW IT MOUNTS: unlike the arm segments this part has no rotary collar. It is
+    a hub that press-fits straight onto the J6 motor's shaft, with its z = 0.005
+    face against the top T-joint's motor plate. Those two mate exactly: the
+    plate's outer face at y = -36.000 spans x +/-30.50 and z 30.50..91.50, i.e. a
+    r = 30.5 circle about (x 0, z 61.000) - the same circle this part's bottom
+    face fits to 0.0 microns.
+    rpy = (pi/2, 0, 0) turns the hub's +Z onto the T-joint's -Y, which is the
+    direction the J6 shaft points, so the hub runs outward from the plate.
+    The part's own bottom sits at z = 0.005 rather than 0, so it stands 5 microns
+    off the plate. That is below the mesh's own precision and is left as authored
+    rather than nudged - the geometry is maintained exactly.
+    FIXED for now, by request. The origin below is already the axis of rotation,
+    so J6's motion is a type change plus an axis and limit.
+  -->
+  <joint name="J6" type="fixed">
+    <parent link="j6_top_t_joint"/>
+    <child  link="gripper_connection"/>
+    <origin xyz="0 ${-36.000 * mm} ${61.000 * mm}" rpy="${pi/2} 0 0"/>
+  </joint>
+  <!--
+    Exact inertia, tetrahedral integration, per unit mass.
+      centre of mass (+0.4702, +0.0977, +11.3558) mm in the mesh frame
+  -->
+  <xacro:property name="gc_ixx_per_kg" value="2.854420869e-04"/>
+  <xacro:property name="gc_iyy_per_kg" value="3.005431716e-04"/>
+  <xacro:property name="gc_izz_per_kg" value="4.641025920e-04"/>
+  <xacro:property name="gc_ixy_per_kg" value="2.735988350e-08"/>
+  <xacro:property name="gc_ixz_per_kg" value="-6.061291888e-06"/>
+  <xacro:property name="gc_iyz_per_kg" value="7.227527713e-07"/>
+  <link name="gripper_connection">
+    <visual>
+      <origin xyz="0 0 0" rpy="0 0 0"/>
+      <geometry>
+        <mesh filename="${mesh_dir}/visual/gripper_connection.stl" scale="${mesh_scale}"/>
+      </geometry>
+      <material name="armold_grey"/>
+    </visual>
+    <collision>
+      <origin xyz="0 0 0" rpy="0 0 0"/>
+      <geometry>
+        <mesh filename="${mesh_dir}/visual/gripper_connection.stl" scale="${mesh_scale}"/>
+      </geometry>
+    </collision>
+    <inertial>
+      <origin xyz="${0.4702 * mm} ${0.0977 * mm} ${11.3558 * mm}" rpy="0 0 0"/>
+      <mass value="${mass_gripper_connection}"/>
+      <inertia
+        ixx="${mass_gripper_connection * gc_ixx_per_kg}" iyy="${mass_gripper_connection * gc_iyy_per_kg}"
+        izz="${mass_gripper_connection * gc_izz_per_kg}" ixy="${mass_gripper_connection * gc_ixy_per_kg}"
+        ixz="${mass_gripper_connection * gc_ixz_per_kg}" iyz="${mass_gripper_connection * gc_iyz_per_kg}"/>
+    </inertial>
+  </link>
+  <!--
+    NEXT: make J6 revolute, then the rest of the gripper.
   -->
 </robot>

File: src/armold_description/urdf/parameters.xacro (robot description, xacro)
@@ -46,4 +46,7 @@
        Mesh solid volume 98 894.2 mm^3 = 98.8942e-6 m^3, x PLA 1240 kg/m^3. -->
   <xacro:property name="mass_j6_top_t_joint" value="0.1226"/>
+  <!-- [ESTIMATE] Gripper connection - the hub that press-fits on the J6 shaft
+       and carries the gripper. Mesh solid volume 58 763.0 mm^3, x PLA 1240. -->
+  <xacro:property name="mass_gripper_connection" value="0.0729"/>
   <!-- ================================================================ -->
   <!-- Motors                                                            -->

Commit message: Change J6 joint type from fixed to revolute with updated axis and limits

File: src/armold_description/urdf/armold.urdf.xacro (robot description, xacro)
@@ -596,5 +596,5 @@
   </xacro:nema17>
   <!-- ================================================================== -->
-  <!-- J6 - carries the gripper connection. STATIC FOR NOW.                 -->
+  <!-- J6 - gripper roll, driven by the 23 mm stepper in the top T-joint   -->
   <!-- ================================================================== -->
   <!--
@@ -617,11 +617,19 @@
     off the plate. That is below the mesh's own precision and is left as authored
     rather than nudged - the geometry is maintained exactly.
-    FIXED for now, by request. The origin below is already the axis of rotation,
-    so J6's motion is a type change plus an axis and limit.
-  -->
-  <joint name="J6" type="fixed">
+    Revolute about the hub's own +Z - the blue axis in RViz. rpy = (pi/2, 0, 0)
+    sends that +Z onto the T-joint's -Y, which is the direction the J6 shaft
+    points, so the axis is the shaft and "0 0 1" in the joint frame says so.
+    This is the same relationship J2 has with the base T-joint, one part family
+    and one pocket design reused at both ends of the arm.
+    LIMITS ARE PROVISIONAL: +/-180 deg placeholder, as for J1-J5. A hub pressed
+    on a bare shaft has no hard stop, so the real limit will come from cabling
+    rather than from geometry.
+  -->
+  <joint name="J6" type="revolute">
     <parent link="j6_top_t_joint"/>
     <child  link="gripper_connection"/>
     <origin xyz="0 ${-36.000 * mm} ${61.000 * mm}" rpy="${pi/2} 0 0"/>
+    <axis xyz="0 0 1"/>
+    <limit lower="${-pi}" upper="${pi}" effort="10.0" velocity="3.14"/>
   </joint>
   <!--

Commit message: Add gripper housing definition with mass parameter to URDF files

File: src/armold_description/urdf/armold.urdf.xacro (robot description, xacro)
@@ -666,6 +666,69 @@
     </inertial>
   </link>
-  <!--
-    NEXT: make J6 revolute, then the rest of the gripper.
+  <!-- ================================================================== -->
+  <!-- Gripper housing - bolted to the connection hub, no relative motion   -->
+  <!-- ================================================================== -->
+  <!--
+    Source mesh : Gripper - Housing.stl  (5558 triangles)
+    Measured    : bbox x +/-25.000, y +/-20.000, z 0.000..25.150
+    MATING, from the two parts alone:
+      footprint   housing's z = 0.250 face spans x +/-25.000, y +/-20.000 with a
+                  max radius of 31.206. The connection's z = 31.905 top face has
+                  exactly the same three numbers. Below z = 0.250 the housing
+                  steps in to +/-24.750 / +/-19.750 - a 0.25 mm lead-in chamfer,
+                  not a spigot.
+      screws      housing has 4 x dia 4.00 bores at (+/-23.000, +/-18.000)
+                  running z 4.5..18.0; the connection has 4 x dia 4.00 at the
+                  SAME (+/-23.000, +/-18.000) near its top.
+    ORIENTATION: note that neither of the above pins it. The +/-25 / +/-20
+    footprint and the (+/-23, +/-18) hole pattern are both symmetric under a
+    180 deg turn about Z, so measurement alone leaves two valid orientations.
+    The correct one is yaw = 180 deg, per the assembly drawing.
+    So: seats on the hub's top face at z = 31.905 mm in the connection's frame,
+    turned 180 deg about Z. Mesh used exactly as authored - the flip lives in
+    the joint, not in the geometry.
+    FIXED, not revolute: the two are bolted together. The gripper's moving parts
+    are the slides and arms inside this housing, which come next.
+  -->
+  <joint name="gripper_housing_fixed" type="fixed">
+    <parent link="gripper_connection"/>
+    <child  link="gripper_housing"/>
+    <origin xyz="0 0 ${31.905 * mm}" rpy="0 0 ${pi}"/>
+  </joint>
+  <!--
+    Exact inertia, tetrahedral integration, per unit mass.
+      centre of mass (+1.4296, -1.4545, +10.8461) mm in the mesh frame
+  -->
+  <xacro:property name="gh_ixx_per_kg" value="1.980362263e-04"/>
+  <xacro:property name="gh_iyy_per_kg" value="3.053506827e-04"/>
+  <xacro:property name="gh_izz_per_kg" value="4.283892400e-04"/>
+  <xacro:property name="gh_ixy_per_kg" value="-3.928712683e-06"/>
+  <xacro:property name="gh_ixz_per_kg" value="6.637863494e-06"/>
+  <xacro:property name="gh_iyz_per_kg" value="4.358863405e-06"/>
+  <link name="gripper_housing">
+    <visual>
+      <origin xyz="0 0 0" rpy="0 0 0"/>
+      <geometry>
+        <mesh filename="${mesh_dir}/visual/gripper_housing.stl" scale="${mesh_scale}"/>
+      </geometry>
+      <material name="armold_grey"/>
+    </visual>
+    <collision>
+      <origin xyz="0 0 0" rpy="0 0 0"/>
+      <geometry>
+        <mesh filename="${mesh_dir}/visual/gripper_housing.stl" scale="${mesh_scale}"/>
+      </geometry>
+    </collision>
+    <inertial>
+      <origin xyz="${1.4296 * mm} ${-1.4545 * mm} ${10.8461 * mm}" rpy="0 0 0"/>
+      <mass value="${mass_gripper_housing}"/>
+      <inertia
+        ixx="${mass_gripper_housing * gh_ixx_per_kg}" iyy="${mass_gripper_housing * gh_iyy_per_kg}"
+        izz="${mass_gripper_housing * gh_izz_per_kg}" ixy="${mass_gripper_housing * gh_ixy_per_kg}"
+        ixz="${mass_gripper_housing * gh_ixz_per_kg}" iyz="${mass_gripper_housing * gh_iyz_per_kg}"/>
+    </inertial>
+  </link>
+  <!--
+    NEXT: the gripper's moving parts - slides, arms and gear inside this housing.
   -->
 </robot>

File: src/armold_description/urdf/parameters.xacro (robot description, xacro)
@@ -49,4 +49,7 @@
        and carries the gripper. Mesh solid volume 58 763.0 mm^3, x PLA 1240. -->
   <xacro:property name="mass_gripper_connection" value="0.0729"/>
+  <!-- [ESTIMATE] Gripper housing - bolted to the connection hub, carries the
+       jaw mechanism. Mesh solid volume 26 134.9 mm^3, x PLA 1240. -->
+  <xacro:property name="mass_gripper_housing" value="0.0324"/>
   <!-- ================================================================ -->
   <!-- Motors                                                            -->
